File: Goom.kicad_pcb (KiCad board)
At the start: 2 copper layers, 69.8 x 100 mm, 80 parts, among them J1 In 1, J2 In 2, J3 CV 1, J4 CV 2, J5 CV 3, J6 Out, J9 Power, Q1 2N3906, Q2 2N3904, Q3 2N3904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

Commit message: clean up
Parts:
- RV5: value 10K Anti-log -> 10K Antilog
Connections:
- U4 pad 1: unconnected-(U4-Pad1) -> (no net)
- U4 pad 5: unconnected-(U4-Pad5) -> (no net)
- U5 pad 1: unconnected-(U5-Pad1) -> (no net)
- U5 pad 5: unconnected-(U5-Pad5) -> (no net)
- U6 pad 1: unconnected-(U6-Pad1) -> (no net)
- U6 pad 5: unconnected-(U6-Pad5) -> (no net)
Routing:
- net Net-(R2-Pad2): track 0.00 -> 7.75 mm
Other:
- board text removed: "Frequency"
- board text removed: "In"
- board text removed: "Resonance"

Commit message: clean up again
Routing:
- net Net-(RN2-R1.2): track 71.4 -> 101.9 mm, vias 1 -> 4
- net Net-(U3A-Q1C): track 88.2 -> 64.1 mm, vias 0 -> 1
- net P3Cb: track 123.0 -> 106.7 mm, vias 1 -> 2
- net Net-(Q1-E): track 63.0 -> 53.7 mm
- net Net-(U3B-Q3B): track 57.4 -> 51.7 mm
- net Out: track 78.4 -> 82.1 mm, vias 0 -> 1
- net P2Ca: track 62.8 -> 59.9 mm
- net Net-(C10-Pad2): track 32.9 -> 34.6 mm
- net Net-(Q1-B): track 189.7 -> 188.2 mm
- net Net-(J9-Pin_10): track 19.1 -> 20.0 mm
- net Net-(U2A-Q2B): track 74.1 -> 74.8 mm
- net P1Ca: track 107.6 -> 108.3 mm
- net P1Cb: track 60.7 -> 61.4 mm
- net Net-(U2A-Q1B): track 40.8 -> 40.2 mm
- net Net-(U3A-Q2C): track 39.9 -> 39.6 mm, vias 1 -> 0
Other:
- board text added: "CRANKERY VCF ONE"
- board text added: "CV 1"
- board text added: "CV 2"
- board text added: "CV 3"
- board text added: "EMPHASIS"
- board text added: "Emphasis"
- board text added: "FREQUENCY"
- board text added: "Frequency"
- board text added: "GOOM"
- board text added: "OUTPUT"
- board text removed: "crankery vcf one"
- board text removed: "cv 1"
- board text removed: "cv 2"
- board text removed: "cv 3"
- board text removed: "emphasis"
- board text removed: "goom vcf"
- board text removed: "output"
